File: mchck.kicad_pcb (KiCad board)
At the start: 2 copper layers, 36.6 x 18.8 mm, 41 parts, among them J3 MICRO_USB, P1 RIGHT_PINS, P10 GND, P11 D-, P12 D+, P2 DEBUG, P3 UPPER_PINS, P4 LOWER_PINS, P5 CHG, P7 LIPO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

Commit message: properly mark R5 rc3 on silk screen
Other:
- board text added: "R5 rc3"
- board text removed: "R5 rc4"
Changed lines of the file:
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@@
   (gr_line (start 69.723 41.91) (end 67.437 41.91) (angle 90) (layer F.SilkS) (width 0.14986))
   (gr_arc (start 73.66 55.753) (end 72.8345 56.5785) (angle 270) (layer F.SilkS) (width 0.14986))
-  (gr_text "R5\nrc4" (at 40 57.1 90) (layer B.SilkS)
+  (gr_text "R5\nrc3" (at 40 57.1 90) (layer B.SilkS)
     (effects (font (size 0.89916 0.89916) (thickness 0.14986)) (justify right mirror))
   )
